File: hardware/tinyups.kicad_pcb (KiCad board)
At the start: 4 copper layers, 147.4 x 92.6 mm, 122 parts, among them J1 XT60, J2 XT30, J3 USB, J4 SWD, J5 FAN, Q1 N-FET 40V, Q10 N-FET 40V, Q11 N-FET 40V, Q12 N-FET 40V, Q2 N-FET 40V, Q3 N-FET 30V, Q4 N-FET 30V, Q5 N-FET 30V, Q6 N-FET 30V, Q7 N-FET 40V, Q8 N-FET 40V, Q9 N-FET 40V, U1 LM5069, U2 LM74700-Q1, U3 BQ25720, U4 LM5176, U5 BQ76942, U6 RP2040, U7 W25Q128, U8 3V3, Y1 12MHz

Commit message: work on routing
Parts:
- moved C18 143.6 mm to (10.7, 124.5)
- moved C16 143.6 mm to (4.72, 124.5)
- moved D4 141.5 mm to (136.4, 108.3)
- moved R43 136.8 mm to (136.2, 54.9)
- moved Q10 123.6 mm to (22.2, 106.5)
- moved Q9 123.6 mm to (8.57, 106.5)
- moved R16 116.0 mm to (16.9, 124.4)
- moved R17 116.0 mm to (23.3, 124.4)
- moved R19 116.0 mm to (29.4, 124.4)
- moved C17 114.7 mm to (8.42, 92.6)
- moved C24 111.6 mm to (137.3, 94.5)
- moved R18 108.8 mm to (42.7, 104.7)
- moved U8 107.6 mm to (131.0, 95.2)
- moved D5 106.0 mm to (100.7, 115.9)
- moved C10 104.6 mm to (11.0, 116.9)
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Other:
- board size 147.4 x 92.6 mm -> 144.6 x 137.5 mm

Commit message: more work on routing
Routing:
- net /SW1: track 0.00 -> 281.0 mm, vias 0 -> 3
- net /+3V3: track 0.00 -> 274.9 mm, vias 0 -> 10
- net /SW2: track 0.00 -> 264.4 mm, vias 0 -> 9
- net /VBAT: track 0.00 -> 234.6 mm, vias 0 -> 9
- net /GND: track 0.00 -> 209.7 mm, vias 0 -> 41
- net /VOUT12: track 0.00 -> 182.3 mm, vias 0 -> 4
- net /I2C_SDA: track 0.00 -> 133.8 mm, vias 0 -> 4
- net /I2C_SCL: track 0.00 -> 132.7 mm, vias 0 -> 4
- net /IN_VALID: track 0.00 -> 114.0 mm, vias 0 -> 3
- net /VIN_LM: track 0.00 -> 60.9 mm, vias 0 -> 4
- net /CELL4: track 0.00 -> 60.4 mm, vias 0 -> 2
- net /CELL0: track 0.00 -> 56.0 mm, vias 0 -> 3
- net /N_ACN: track 0.00 -> 53.4 mm, vias 0 -> 3
- net /N_USBDP_C: track 0.00 -> 53.2 mm, vias 0 -> 1
- net /N_CS: track 0.00 -> 52.1 mm, vias 0 -> 3
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- added copper zone on In1.Cu, net /GND
- added copper zone on In2.Cu, net /VIN_SYS
