File: hardware/tinyups.kicad_pcb (KiCad board)
At the start: 4 copper layers, 150 x 140 mm, 124 parts

Commit message: new terminal power rating metric, new FET selection
Parts:
- 1Q1, 3Q1, 4Q1, 4Q2: value N-FET 40V -> NTMFS5C410N; footprint Package_TO_SOT_SMD:TO-252-2 -> Package_SON:VSONP-8-1EP_5x6_P1.27mm
- 2Q1, 2Q2, 2Q3, 2Q4: value N-FET 30V -> NTMFS4C01N; footprint Package_TO_SOT_SMD:TO-252-2 -> Package_SON:VSONP-8-1EP_5x6_P1.27mm
- 5Q1, 5Q2, 5Q3, 5Q4: value N-FET 40V -> NTMFS5C430N; footprint Package_TO_SOT_SMD:TO-252-2 -> Package_SON:VSONP-8-1EP_5x6_P1.27mm
Connections:
- 1Q1 pad 1: /N_GATE -> /VIN_SYS
- 1Q1 pad 2: /VIN_SYS -> /N_GATE
- 2Q1 pad 1: /N_G3 -> /SW1
- 2Q1 pad 2: /SW1 -> /N_G3
- 2Q2 pad 1: /N_G4 -> /GND
- 2Q2 pad 2: /GND -> /N_G4
- 2Q3 pad 1: /N_G5 -> /GND
- 2Q3 pad 2: /GND -> /N_G5
- 2Q4 pad 1: /N_G6 -> /SW2
- 2Q4 pad 2: /SW2 -> /N_G6
- 3Q1 pad 1: /N_PGATE -> /VBAT
- 3Q1 pad 2: /VBAT -> /N_PGATE
- 4Q1 pad 1: /N_CHG -> /N_PACKMID
- 4Q1 pad 2: /N_PACKMID -> /N_CHG
- 4Q2 pad 1: /N_DSG -> /N_PACKMID
- 4Q2 pad 2: /N_PACKMID -> /N_DSG
- 5Q1 pad 1: /N_G7 -> /SW1_OUT
- 5Q1 pad 2: /SW1_OUT -> /N_G7
- 5Q2 pad 1: /N_G8 -> /N_CS
- 5Q2 pad 2: /N_CS -> /N_G8
- 5Q3 pad 1: /N_G9 -> /N_CS
- 5Q3 pad 2: /N_CS -> /N_G9
- 5Q4 pad 1: /N_G10 -> /SW2_OUT
- 5Q4 pad 2: /SW2_OUT -> /N_G10
Routing:
- added copper zone on F.Cu, net /CELL0
- added copper zone on F.Cu, net /N_ACN
- added copper zone on F.Cu, net /N_CS
- added copper zone on F.Cu, net /N_PACKMID
- added copper zone on F.Cu, net /PACK+
- added copper zone on F.Cu, net /VBUS
- added copper zone on F.Cu, net /VIN_LM

Commit message: board fixup, added shunt sense gate
Connections:
- 2R1 pad 1: /VBUS -> /VIN_SYS
- 2U1 pad 1: /VBUS -> /VIN_SYS
- 2U1 pad 3: /VBUS -> /VIN_SYS
Changed lines of the file:
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@@
 			(size 3.94 5.84)
 			(layers "F.Cu" "F.Mask" "F.Paste")
-			(net 29 "/VBUS")
+			(net 6 "/VIN_SYS")
 		)
 		(pad "2" smd rect
@@
 			(size 0.129289 0.129289)
 			(layers "F.Cu" "F.Mask" "F.Paste")
-			(net 29 "/VBUS")
+			(net 6 "/VIN_SYS")
 			(options
 				(clearance outline)
@@
 			(layers "F.Cu" "F.Mask" "F.Paste")
 			(roundrect_rratio 0.25)
-			(net 29 "/VBUS")
+			(net 6 "/VIN_SYS")
 		)
 		(pad "4" smd roundrect

Commit message: auto-work on resume
Parts:
- moved 6C4 156.5 mm to (130.0, 9.80), turned to 0 degrees
- moved 6J3 151.3 mm to (144.4, 11.9)
- moved 6R6 150.0 mm to (138.4, 12.1)
- moved 6R7 143.8 mm to (138.0, 8.89)
- moved 6R1 139.2 mm to (131.8, 34.8)
- moved 6C5 137.8 mm to (126.5, 35.1)
- moved 6J4 135.3 mm to (144.8, 26.1)
- moved 6C1 132.8 mm to (119.3, 37.8), turned to 180 degrees
- moved 6D1 132.8 mm to (109.3, 29.2), turned to 0 degrees
- moved 6R2 130.1 mm to (113.2, 28.9), turned to 180 degrees
- moved 6U2 128.9 mm to (122.1, 10.3)
- moved 6U1 128.6 mm to (124.0, 28.6)
- moved 6Y1 126.9 mm to (122.7, 41.6), turned to 0 degrees
- moved 6C2 124.9 mm to (125.5, 37.7), turned to 0 degrees
- moved 6R8 121.5 mm to (119.6, 23.3), turned to 0 degrees
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Routing:
- removed copper zone on F.Cu, net /VBUS

Commit message: add part proximity metrics
Parts:
- moved 5C1 43.1 mm to (112.0, 69.9), turned to 0 degrees
- moved 3C3 40.8 mm to (100.6, 57.9)
- moved 3C2 39.3 mm to (109.5, 62.8), turned to 90 degrees
- moved 6C3 20.5 mm to (110.9, 49.4), turned to 0 degrees

Commit message: (incomplete) voronoi pour overlap resolution
Parts:
- moved 5C9 6.29 mm to (115.9, 120.1)
- moved 4Q1 6.13 mm to (47.1, 46.5)
- moved 3C2 0.17 mm to (109.4, 63.0)
Routing:
- added copper zone on F.Cu, net /GND
