File: hardware/tinyups.kicad_sch (KiCad schematic)
At the start: 110 parts, among them J1 XT60, J2 XT30, J3 USB, J4 SWD, J5 FAN, Q1 N-FET 40V, Q10 N-FET 40V, Q11 N-FET 40V, Q12 N-FET 40V, Q2 N-FET 40V, Q3 N-FET 30V, Q4 N-FET 30V, Q5 N-FET 30V, Q6 N-FET 30V, Q7 N-FET 40V, Q8 N-FET 40V, Q9 N-FET 40V, U1 LM5069, U2 LM74700-Q1, U3 BQ25720, U4 LM5176, U5 BQ76942, U6 RP2040, U7 W25Q128, U8 3V3, Y1 12MHz

Commit message: more work on hardware, routing
Parts:
- added C29: 10n, Capacitor_SMD:C_0805_2012Metric, symbol Device:C
- added C30: 1n, Capacitor_SMD:C_0805_2012Metric, symbol Device:C
- added C31, C32, C33: 100n, Capacitor_SMD:C_0805_2012Metric, symbol Device:C
- added R40, R41, R42, R43, R44: 10k, Resistor_SMD:R_0805_2012Metric, symbol Device:R
- added R45, R46: 100k, Resistor_SMD:R_0805_2012Metric, symbol Device:R
- C1, C10, C11, C12, C13, C14, C15, C16, C18, C19, C2, C20, C21, C22, C23, C24, C25, C26, C27, C28, C5, C6, C7, C8, C9, Cf0, Cf1, Cf2, Cf3, Cf4: footprint (none) -> Capacitor_SMD:C_0805_2012Metric
- C17, C3, C4: footprint (none) -> Capacitor_SMD:CP_Elec_8x10
- D1: footprint (none) -> Diode_SMD:D_SMB
- D2, D3, D4, D5: footprint (none) -> LED_SMD:LED_0805_2012Metric
- F1: footprint (none) -> Fuse:Fuse_1206_3216Metric
- J1: footprint (none) -> Connector_Wire:SolderWire-2.5sqmm_1x02_P8.8mm_D2.4mm_OD4.4mm
- J2: footprint (none) -> Connector_Wire:SolderWire-2.5sqmm_1x02_P7.2mm_D2.4mm_OD3.6mm
- J3, J4: footprint (none) -> Connector_PinHeader_2.54mm:PinHeader_1x03_P2.54mm_Vertical
- J5: footprint (none) -> Connector_PinHeader_2.54mm:PinHeader_1x04_P2.54mm_Vertical
- L2, L3: footprint (none) -> Inductor_SMD:L_12x12mm_H8mm
- Q1, Q10, Q11, Q12, Q2, Q3, Q4, Q5, Q6, Q7, Q8, Q9: footprint (none) -> Package_TO_SOT_SMD:TO-252-2
- R1, R10, R18, R25, R9: footprint (none) -> Resistor_SMD:R_2512_6332Metric
- R11, R12, R13, R14, R15, R16, R17, R19, R2, R20, R21, R22, R23, R24, R26, R27, R28, R29, R3, R30, R31, R32, R33, R34, R35, R36, R37, R38, R4, R5, R6, R7, R8, Rf0, Rf1, Rf2, Rf3, Rf4: footprint (none) -> Resistor_SMD:R_0805_2012Metric
- U1: footprint (none) -> Package_SO:VSSOP-10_3x3mm_P0.5mm
- U2: footprint (none) -> Package_TO_SOT_SMD:SOT-23-6
- U3: footprint (none) -> Package_DFN_QFN:QFN-32-1EP_4x4mm_P0.4mm_EP2.65x2.65mm
- U4: footprint (none) -> Package_DFN_QFN:QFN-28-1EP_4x4mm_P0.4mm_EP2.4x2.4mm
- U5: footprint (none) -> Package_QFP:TQFP-48_7x7mm_P0.5mm
- U6: footprint (none) -> Package_DFN_QFN:QFN-56-1EP_7x7mm_P0.4mm_EP3.2x3.2mm
- U7: footprint (none) -> Package_SO:SOIC-8_3.9x4.9mm_P1.27mm
- U8: footprint (none) -> Package_TO_SOT_SMD:SOT-23-5
- Y1: footprint (none) -> Crystal:Crystal_SMD_5032-2Pin_5.0x3.2mm
Connections:
- net +3V3: now also R43.2, R44.2
- net GND: now also U3.14 (CMPIN), U3.5 (OTG/VAP/FRS), C29.2, C30.2, C31.2, C32.2, C33.2
- net N_REG1: now also R45.2, R46.2
- net N_PSYS: now reaches U3.10 (PSYS)
- net N_PSYS: now also C31.1
- net N_PROCHOT: now reaches U3.11 (PROCHOT)
- net N_PROCHOT: now also R44.1
- net N_COMP1: now reaches U3.16 (COMP1)
- net N_COMP1: now also R40.1
- net N_COMP2: now reaches U3.17 (COMP2)
- net N_COMP2: now also C30.1
- net N_CHGOK: now reaches U3.4 (CHRG_OK)
- net N_CHGOK: now also R43.1
- net N_IADPT: now reaches U3.8 (IADPT)
- net N_IADPT: now also R41.1
- net N_IBAT: now reaches U3.9 (IBAT)
- net N_IBAT: now also R42.1
- net N_CFETOFF: now reaches U5.29 (CFETOFF)
- net N_CFETOFF: now also R45.1
- net N_DFETOFF: now reaches U5.30 (DFETOFF)
- net N_DFETOFF: now also R46.1
- new net N_COMP1B: C29.1, R40.2
- new net N_IADPTB: C32.1, R41.2
- new net N_IBATB: C33.1, R42.2
- no-connect marks 51 -> 40

Commit message: more work on routing
Connections:
- net SW1: no longer C10.2, L3.1, Q7.2 (S), Q8.3 (D), U4.25 (SW1)
- net SW2: no longer C11.2, L3.2, Q10.2 (S), Q9.3 (D), U4.15 (SW2)
- new net SW1_OUT: C10.2, L3.1, Q7.2 (S), Q8.3 (D), U4.25 (SW1)
- new net SW2_OUT: C11.2, L3.2, Q10.2 (S), Q9.3 (D), U4.15 (SW2)
Changed lines of the file:
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@@
     (effects (font (size 1.27 1.27)))
   )
-  (label "SW1" (at 345.44 54.61 0)
+  (label "SW1_OUT" (at 345.44 54.61 0)
     (effects (font (size 1.27 1.27)))
   )
-  (label "SW1" (at 332.74 101.6 0)
+  (label "SW1_OUT" (at 332.74 101.6 0)
     (effects (font (size 1.27 1.27)))
   )
-  (label "SW1" (at 358.14000000000004 91.44 0)
+  (label "SW1_OUT" (at 358.14000000000004 91.44 0)
     (effects (font (size 1.27 1.27)))
   )
-  (label "SW1" (at 368.3 118.11 0)
+  (label "SW1_OUT" (at 368.3 118.11 0)
     (effects (font (size 1.27 1.27)))
   )
-  (label "SW1" (at 304.8 125.73 0)
+  (label "SW1_OUT" (at 304.8 125.73 0)
     (effects (font (size 1.27 1.27)))
   )
-  (label "SW2" (at 345.44 29.209999999999997 0)
+  (label "SW2_OUT" (at 345.44 29.209999999999997 0)
     (effects (font (size 1.27 1.27)))
   )
-  (label "SW2" (at 383.54 91.44 0)
+  (label "SW2_OUT" (at 383.54 91.44 0)
     (effects (font (size 1.27 1.27)))
   )
-  (label "SW2" (at 408.94 101.6 0)
+  (label "SW2_OUT" (at 408.94 101.6 0)
     (effects (font (size 1.27 1.27)))
   )
-  (label "SW2" (at 368.3 125.73 0)
+  (label "SW2_OUT" (at 368.3 125.73 0)
     (effects (font (size 1.27 1.27)))
   )
-  (label "SW2" (at 330.2 125.73 0)
+  (label "SW2_OUT" (at 330.2 125.73 0)
     (effects (font (size 1.27 1.27)))
   )

Commit message: work on routing. llm hit wall
Other:
- company, title: (none) -> TinyUPS
Changed lines of the file:
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@@
 (kicad_sch (version 20211014) (generator kiutils)
-  (paper "A4")
+  (paper "A1")
+  (title_block
+    (title "TinyUPS")
+    (date "2026-10-12")
+    (rev "0.1")
+    (company "TinyUPS")
+  )
   (no_connect (at 175.26 62.230000000000004))
   (no_connect (at 205.74 36.83))

Commit message: quantify power components, placement, add render for inspection
Parts:
- added J6: PACK, Connector_Wire:SolderWire-2.5sqmm_1x02_P8.8mm_D2.4mm_OD4.4mm, symbol Connector_Generic:Conn_01x02
- added J7: CELLS, Connector_PinHeader_2.54mm:PinHeader_1x05_P2.54mm_Vertical, symbol Connector_Generic:Conn_01x05
Connections:
- net N_CATH is gone; now on net VIN_SYS: Q2.3 (D), U2.4 (CATHODE)
- net CELL0: now also J6.2 (Pin_2), J7.1 (Pin_1)
- net CELL1: now also J7.2 (Pin_2)
- net CELL2: now also J7.3 (Pin_3)
- net CELL3: now also J7.4 (Pin_4)
- net CELL4: now also J7.5 (Pin_5)
- net N_PACKMID: now also Q12.2 (S); no longer Q12.3 (D)
- net VBAT: now also Q12.3 (D); no longer C22.1, C23.2, Q11.3 (D), Q12.2 (S), U5.36 (REGIN), U5.47 (BAT)
- new net PACK+: C22.1, C23.2, J6.1 (Pin_1), Q11.3 (D), U5.36 (REGIN), U5.47 (BAT)
Changed lines of the file:
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@@
     (effects (font (size 1.27 1.27)))
   )
-  (label "N_CATH" (at 54.61 124.46000000000001 0)
+  (label "VIN_SYS" (at 54.61 124.46000000000001 0)
     (effects (font (size 1.27 1.27)))
   )
@@
     (effects (font (size 1.27 1.27)))
   )
-  (label "N_CATH" (at 66.04 116.84 0)
+  (label "VIN_SYS" (at 66.04 116.84 0)
     (effects (font (size 1.27 1.27)))
   )
@@
     (effects (font (size 1.27 1.27)))
   )
+  (label "PACK+" (at 553.7199999999999 96.52 0)
+    (effects (font (size 1.27 1.27)))
+  )
+  (label "CELL0" (at 553.7199999999999 99.06 0)
+    (effects (font (size 1.27 1.27)))
+  )
+  (label "CELL0" (at 579.12 91.44 0)
+    (effects (font (size 1.27 1.27)))
+  )
+  (label "CELL1" (at 579.12 93.97999999999999 0)
+    (effects (font (size 1.27 1.27)))
+  )
+  (label "CELL2" (at 579.12 96.52 0)
+    (effects (font (size 1.27 1.27)))
+  )
+  (label "CELL3" (at 579.12 99.06 0)
+    (effects (font (size 1.27 1.27)))
+  )
+  (label "CELL4" (at 579.12 101.6 0)
+    (effects (font (size 1.27 1.27)))
+  )
   (label "CELL0" (at 304.8 219.71 0)
     (effects (font (size 1.27 1.27)))
@@
     (effects (font (size 1.27 1.27)))
   )
-  (label "VBAT" (at 497.84000000000003 44.45 0)
+  (label "PACK+" (at 497.84000000000003 44.45 0)
     (effects (font (size 1.27 1.27)))
   )
-  (label "VBAT" (at 508.0 168.91 0)
+  (label "PACK+" (at 508.0 168.91 0)
     (effects (font (size 1.27 1.27)))
   )
@@
     (effects (font (size 1.27 1.27)))
   )
-  (label "VBAT" (at 497.84000000000003 72.39 0)
+  (label "PACK+" (at 497.84000000000003 72.39 0)
     (effects (font (size 1.27 1.27)))
   )
@@
     (effects (font (size 1.27 1.27)))
   )
-  (label "VBAT" (at 434.34000000000003 116.84 0)
+  (label "PACK+" (at 434.34000000000003 116.84 0)
     (effects (font (size 1.27 1.27)))
   )
-  (label "VBAT" (at 459.74 127.0 0)
+  (label "VBAT" (at 459.74 116.84 0)
     (effects (font (size 1.27 1.27)))
   )
@@
     (effects (font (size 1.27 1.27)))
   )
-  (label "N_PACKMID" (at 459.74 116.84 0)
+  (label "N_PACKMID" (at 459.74 127.0 0)
     (effects (font (size 1.27 1.27)))
   )
-  (label "VBAT" (at 533.4 176.53 0)
+  (label "PACK+" (at 533.4 176.53 0)
     (effects (font (size 1.27 1.27)))
   )
@@
         )
       )
+    )
+  )
+  (symbol (lib_id "Connector_Generic:Conn_01x02") (at 558.8 96.52 0) (unit 1)
+    (in_bom yes) (on_board yes) (dnp no)
+    (property "Reference" "J6" (at 561.3399999999999 93.97999999999999 0)
+      (effects (font (size 1.27 1.27)))
+    )
+    (property "Value" "PACK" (at 561.3399999999999 99.06 0)
+      (effects (font (size 1.27 1.27)))
+    )
+    (property "Footprint" "Connector_Wire:SolderWire-2.5sqmm_1x02_P8.8mm_D2.4mm_OD4.4mm" (at 558.8 96.52 0)
+      (effects (font (size 1.0 1.0)) hide)
+    )
+    (property "Datasheet" "~" (at 558.8 96.52 0)
+      (effects (font (size 1.0 1.0)) hide)
+    )
+    (pin "1")
+    (pin "2")
+    (instances
+      (project "tinyups"
+        (path "/"
+          (reference "J6") (unit 1)
+        )
+      )
+    )
+  )
+  (symbol (lib_id "Connector_Generic:Conn_01x05") (at 584.2 96.52 0) (unit 1)
+    (in_bom yes) (on_board yes) (dnp no)
+    (property "Reference" "J7" (at 586.74 93.97999999999999 0)
+      (effects (font (size 1.27 1.27)))
+    )
+    (property "Value" "CELLS" (at 586.74 99.06 0)
+      (effects (font (size 1.27 1.27)))
+    )
+    (property "Footprint" "Connector_PinHeader_2.54mm:PinHeader_1x05_P2.54mm_Vertical" (at 584.2 96.52 0)
+      (effects (font (size 1.0 1.0)) hide)
+    )
+    (property "Datasheet" "~" (at 584.2 96.52 0)
+      (effects (font (size 1.0 1.0)) hide)
+    )
+    (pin "1")
+    (pin "2")
+    (pin "3")
+    (pin "4")
+    (pin "5")
+    (instances
+      (project "tinyups"
+        (path "/"
+          (reference "J7") (unit 1)
+        )
+      )

Commit message: try to find a new placement approach
Parts:
- removed C1: TBD, Capacitor_SMD:C_0805_2012Metric, symbol Device:C
- removed C10, C11, C2, C23, C31, C32, C33, Cf0, Cf1, Cf2, Cf3, Cf4: 100n, Capacitor_SMD:C_0805_2012Metric, symbol Device:C
- removed C12, C29: 10n, Capacitor_SMD:C_0805_2012Metric, symbol Device:C
- removed C13, C14, C15, C30: 1n, Capacitor_SMD:C_0805_2012Metric, symbol Device:C
- removed C16, C19, C20, C21, C22, C28, C7, C8: 1u, Capacitor_SMD:C_0805_2012Metric, symbol Device:C
- removed C17: 220u, Capacitor_SMD:CP_Elec_8x10, symbol Device:C
- removed C18, C26, C27, C9: 10u, Capacitor_SMD:C_0805_2012Metric, symbol Device:C
- removed C24, C25: 20p, Capacitor_SMD:C_0805_2012Metric, symbol Device:C
- removed C3, C4: 470u, Capacitor_SMD:CP_Elec_8x10, symbol Device:C
- removed C5, C6: 47n, Capacitor_SMD:C_0805_2012Metric, symbol Device:C
- removed D1: SMBJ15A, Diode_SMD:D_SMB, symbol Device:D_TVS
- removed D2, D3, D4, D5: LED, LED_SMD:LED_0805_2012Metric, symbol Device:LED
- removed F1: 25A, Fuse:Fuse_1206_3216Metric, symbol Device:Fuse
- removed J1: XT60, Connector_Wire:SolderWire-2.5sqmm_1x02_P8.8mm_D2.4mm_OD4.4mm, symbol Connector_Generic:Conn_01x02
- removed J2: XT30, Connector_Wire:SolderWire-2.5sqmm_1x02_P7.2mm_D2.4mm_OD3.6mm, symbol Connector_Generic:Conn_01x02
- removed J3: USB, Connector_PinHeader_2.54mm:PinHeader_1x03_P2.54mm_Vertical, symbol Connector_Generic:Conn_01x03
- removed J4: SWD, Connector_PinHeader_2.54mm:PinHeader_1x03_P2.54mm_Vertical, symbol Connector_Generic:Conn_01x03
- removed J5: FAN, Connector_PinHeader_2.54mm:PinHeader_1x04_P2.54mm_Vertical, symbol Connector_Generic:Conn_01x04
- removed J6: PACK, Connector_Wire:SolderWire-2.5sqmm_1x02_P8.8mm_D2.4mm_OD4.4mm, symbol Connector_Generic:Conn_01x02
- removed J7: CELLS, Connector_PinHeader_2.54mm:PinHeader_1x05_P2.54mm_Vertical, symbol Connector_Generic:Conn_01x05
- removed L2: 2.2u, Inductor_SMD:L_12x12mm_H8mm, symbol Device:L
- removed L3: 1u0, Inductor_SMD:L_12x12mm_H8mm, symbol Device:L
- removed Q1, Q10, Q11, Q12, Q2, Q7, Q8, Q9: N-FET 40V, Package_TO_SOT_SMD:TO-252-2, symbol Transistor_FET:Q_NMOS_GSD
- removed Q3, Q4, Q5, Q6: N-FET 30V, Package_TO_SOT_SMD:TO-252-2, symbol Transistor_FET:Q_NMOS_GSD
- removed R1: 2.2m, Resistor_SMD:R_2512_6332Metric, symbol Device:R
- removed R10, R9: 5m, Resistor_SMD:R_2512_6332Metric, symbol Device:R
- removed R11, R12, R16, R22, R24, R29, R30, R45, R46, R8: 100k, Resistor_SMD:R_0805_2012Metric, symbol Device:R
- removed R13, R14, R15, R21, R23, R38, R40, R41, R42, R43, R44: 10k, Resistor_SMD:R_0805_2012Metric, symbol Device:R
- removed R17: 7k15, Resistor_SMD:R_0805_2012Metric, symbol Device:R
- removed R18, R25: 1m, Resistor_SMD:R_2512_6332Metric, symbol Device:R
- removed R19: 27k, Resistor_SMD:R_0805_2012Metric, symbol Device:R
- removed R2: TBD-UV-hi, Resistor_SMD:R_0805_2012Metric, symbol Device:R
- removed R20: 93k1, Resistor_SMD:R_0805_2012Metric, symbol Device:R
- removed R26, R27, R28: 10k-NTC, Resistor_SMD:R_0805_2012Metric, symbol Device:R
- removed R3: TBD-UV-lo, Resistor_SMD:R_0805_2012Metric, symbol Device:R
- removed R31, R32, R33, R34, R35: 1k, Resistor_SMD:R_0805_2012Metric, symbol Device:R
- removed R36, R37: 27, Resistor_SMD:R_0805_2012Metric, symbol Device:R
- removed R4: TBD-OV-hi, Resistor_SMD:R_0805_2012Metric, symbol Device:R
- removed R5: TBD-OV-lo, Resistor_SMD:R_0805_2012Metric, symbol Device:R
- removed R6: TBD-PWR, Resistor_SMD:R_0805_2012Metric, symbol Device:R
- removed R7: 100k-PGD, Resistor_SMD:R_0805_2012Metric, symbol Device:R
- removed Rf0, Rf1, Rf2, Rf3, Rf4: 100, Resistor_SMD:R_0805_2012Metric, symbol Device:R
- removed U1: LM5069, Package_SO:VSSOP-10_3x3mm_P0.5mm, symbol tinyups:LM5069
- removed U2: LM74700-Q1, Package_TO_SOT_SMD:SOT-23-6, symbol tinyups:LM74700-Q1
- removed U3: BQ25720, Package_DFN_QFN:QFN-32-1EP_4x4mm_P0.4mm_EP2.65x2.65mm, symbol tinyups:BQ25720
- removed U4: LM5176, Package_DFN_QFN:QFN-28-1EP_4x4mm_P0.4mm_EP2.4x2.4mm, symbol tinyups:LM5176
- removed U5: BQ76942, Package_QFP:TQFP-48_7x7mm_P0.5mm, symbol tinyups:BQ76942
- removed U6: RP2040, Package_DFN_QFN:QFN-56-1EP_7x7mm_P0.4mm_EP3.2x3.2mm, symbol tinyups:RP2040
- removed U7: W25Q128, Package_SO:SOIC-8_3.9x4.9mm_P1.27mm, symbol tinyups:W25Q128
- removed U8: 3V3, Package_TO_SOT_SMD:SOT-23-5, symbol tinyups:REG_3V3
- removed Y1: 12MHz, Crystal:Crystal_SMD_5032-2Pin_5.0x3.2mm, symbol Device:Crystal
- added 1C1: TBD, Capacitor_SMD:C_0805_2012Metric, symbol Device:C
- added 1D1: SMBJ15A, Diode_SMD:D_SMB, symbol Device:D_TVS
- added 1F1: 25A, Fuse:Fuse_1206_3216Metric, symbol Device:Fuse
- added 1J1: XT60, Connector_Wire:SolderWire-2.5sqmm_1x02_P8.8mm_D2.4mm_OD4.4mm, symbol Connector_Generic:Conn_01x02
- added 1Q1, 3Q1, 4Q1, 4Q2, 5Q1, 5Q2, 5Q3, 5Q4: N-FET 40V, Package_TO_SOT_SMD:TO-252-2, symbol Transistor_FET:Q_NMOS_GSD
- added 1R1: 2.2m, Resistor_SMD:R_2512_6332Metric, symbol Device:R
- added 1R2: TBD-UV-hi, Resistor_SMD:R_0805_2012Metric, symbol Device:R
- added 1R3: TBD-UV-lo, Resistor_SMD:R_0805_2012Metric, symbol Device:R
- added 1R4: TBD-OV-hi, Resistor_SMD:R_0805_2012Metric, symbol Device:R
- added 1R5: TBD-OV-lo, Resistor_SMD:R_0805_2012Metric, symbol Device:R
- added 1R6: TBD-PWR, Resistor_SMD:R_0805_2012Metric, symbol Device:R
- added 1R7: 100k-PGD, Resistor_SMD:R_0805_2012Metric, symbol Device:R
- added 1U1: LM5069, Package_SO:VSSOP-10_3x3mm_P0.5mm, symbol tinyups:LM5069
- added 2C1, 2C2: 47n, Capacitor_SMD:C_0805_2012Metric, symbol Device:C
- added 2C3, 2C4, 4C1, 4C2, 4C3, 4C4, 5C8, 6C5: 1u, Capacitor_SMD:C_0805_2012Metric, symbol Device:C
- added 2C5, 5C4: 10n, Capacitor_SMD:C_0805_2012Metric, symbol Device:C
- added 2C6, 5C5, 5C6, 5C7: 1n, Capacitor_SMD:C_0805_2012Metric, symbol Device:C
- added 2C7, 2C8, 2C9, 3C1, 4C10, 4C5, 4C6, 4C7, 4C8, 4C9, 5C2, 5C3: 100n, Capacitor_SMD:C_0805_2012Metric, symbol Device:C
- added 2L1: 2.2u, Inductor_SMD:L_12x12mm_H8mm, symbol Device:L
- added 2Q1, 2Q2, 2Q3, 2Q4: N-FET 30V, Package_TO_SOT_SMD:TO-252-2, symbol Transistor_FET:Q_NMOS_GSD
- added 2R1, 2R2: 5m, Resistor_SMD:R_2512_6332Metric, symbol Device:R
- added 2R10, 2R11, 2R12, 2R5, 2R6, 2R7, 2R8, 2R9, 5R6, 5R8, 6R8: 10k, Resistor_SMD:R_0805_2012Metric, symbol Device:R
- added 2R3, 2R4, 3R1, 4R5, 4R6, 4R7, 4R8, 5R1, 5R7, 5R9: 100k, Resistor_SMD:R_0805_2012Metric, symbol Device:R
- added 2U1: BQ25720, Package_DFN_QFN:QFN-32-1EP_4x4mm_P0.4mm_EP2.65x2.65mm, symbol tinyups:BQ25720
- added 3C2, 3C3: 470u, Capacitor_SMD:CP_Elec_8x10, symbol Device:C
- added 3U1: LM74700-Q1, Package_TO_SOT_SMD:SOT-23-6, symbol tinyups:LM74700-Q1
- added 4J6: PACK, Connector_Wire:SolderWire-2.5sqmm_1x02_P8.8mm_D2.4mm_OD4.4mm, symbol Connector_Generic:Conn_01x02
- added 4J7: CELLS, Connector_PinHeader_2.54mm:PinHeader_1x05_P2.54mm_Vertical, symbol Connector_Generic:Conn_01x05
- added 4R1, 5R3: 1m, Resistor_SMD:R_2512_6332Metric, symbol Device:R
- added 4R10, 4R11, 4R12, 4R13, 4R9: 100, Resistor_SMD:R_0805_2012Metric, symbol Device:R
- added 4R2, 4R3, 4R4: 10k-NTC, Resistor_SMD:R_0805_2012Metric, symbol Device:R
- added 4U1: BQ76942, Package_QFP:TQFP-48_7x7mm_P0.5mm, symbol tinyups:BQ76942
- added 5C1, 5C10, 6C3, 6C4: 10u, Capacitor_SMD:C_0805_2012Metric, symbol Device:C
- added 5C9: 220u, Capacitor_SMD:CP_Elec_8x10, symbol Device:C
- added 5J2: XT30, Connector_Wire:SolderWire-2.5sqmm_1x02_P7.2mm_D2.4mm_OD3.6mm, symbol Connector_Generic:Conn_01x02
- added 5L1: 1u0, Inductor_SMD:L_12x12mm_H8mm, symbol Device:L
- added 5R2: 7k15, Resistor_SMD:R_0805_2012Metric, symbol Device:R
- added 5R4: 27k, Resistor_SMD:R_0805_2012Metric, symbol Device:R
- added 5R5: 93k1, Resistor_SMD:R_0805_2012Metric, symbol Device:R
- added 5U1: LM5176, Package_DFN_QFN:QFN-28-1EP_4x4mm_P0.4mm_EP2.4x2.4mm, symbol tinyups:LM5176
- added 6C1, 6C2: 20p, Capacitor_SMD:C_0805_2012Metric, symbol Device:C
- added 6D1, 6D2, 6D3, 6D4: LED, LED_SMD:LED_0805_2012Metric, symbol Device:LED
- added 6J3: USB, Connector_PinHeader_2.54mm:PinHeader_1x03_P2.54mm_Vertical, symbol Connector_Generic:Conn_01x03
- added 6J4: SWD, Connector_PinHeader_2.54mm:PinHeader_1x03_P2.54mm_Vertical, symbol Connector_Generic:Conn_01x03
- added 6J5: FAN, Connector_PinHeader_2.54mm:PinHeader_1x04_P2.54mm_Vertical, symbol Connector_Generic:Conn_01x04
- added 6R1, 6R2, 6R3, 6R4, 6R5: 1k, Resistor_SMD:R_0805_2012Metric, symbol Device:R
- added 6R6, 6R7: 27, Resistor_SMD:R_0805_2012Metric, symbol Device:R
- added 6U1: RP2040, Package_DFN_QFN:QFN-56-1EP_7x7mm_P0.4mm_EP3.2x3.2mm, symbol tinyups:RP2040
- added 6U2: W25Q128, Package_SO:SOIC-8_3.9x4.9mm_P1.27mm, symbol tinyups:W25Q128
- added 6U3: 3V3, Package_TO_SOT_SMD:SOT-23-5, symbol tinyups:REG_3V3
- added 6Y1: 12MHz, Crystal:Crystal_SMD_5032-2Pin_5.0x3.2mm, symbol Device:Crystal
Connections:
- net +12V_IN: now also 1F1.1, 1J1.1 (Pin_1), 1R7.1
- net +3V3: now also 2R11.2, 2R12.2, 2R6.2, 2R7.2, 4R5.2, 5R9.2, 6C4.1, 6R1.2, 6R8.2, 6U1.1 (IOVDD), 6U1.10 (IOVDD), 6U1.22 (IOVDD), 6U1.33 (IOVDD), 6U1.42 (IOVDD), 6U1.43 (ADC_AVDD), 6U1.44 (VREG_VIN), 6U1.48 (USB_VDD), 6U1.49 (IOVDD), 6U1.56 (IOVDD), 6U2.7 (VCC), 6U3.4 (VOUT)
- net CELL0: now also 4C7.2, 4J6.2 (Pin_2), 4J7.1 (Pin_1), 4R1.1, 4R9.1, 4U1.18 (SRP)
- net CELL1: now also 4C8.2, 4J7.2 (Pin_2), 4R10.1
- net CELL2: now also 4C9.2, 4J7.3 (Pin_3), 4R11.1
- net CELL3: now also 4C10.2, 4J7.4 (Pin_4), 4R12.1
- net CELL4: now also 4J7.5 (Pin_5), 4R13.1, 4U1.10 (VC5), 4U1.2 (VC9), 4U1.4 (VC8), 4U1.48 (VC10), 4U1.6 (VC7), 4U1.8 (VC6)
- net GND: now also 1C1.2, 1D1.2 (A2), 1J1.2 (Pin_2), 1R3.2, 1R5.2, 1R6.2, 1U1.5 (GND), 2C3.2, 2C4.2, 2C5.2, 2C6.2, 2C7.2, 2C8.2, 2C9.2, 2Q2.2 (S), 2Q3.2 (S), 2R4.2, 2R5.2, 2U1.14 (CMPIN), 2U1.27 (PGND), 2U1.5 (OTG/VAP/FRS), 3C2.2, 3C3.2, 3R1.2, 3U1.2 (GND), 4C1.2, 4C2.2, 4C3.2, 4C4.2, 4C6.2, 4R1.2, 4R2.2, 4R3.2, 4R4.2, 4R6.2, 4U1.17 (VSS), 4U1.20 (SRN), 5C1.2, 5C10.2, 5C4.2, 5C5.2, 5C6.2, 5C7.2, 5C8.2, 5C9.2, 5J2.2 (Pin_2), 5R2.2, 5R3.2, 5R4.2, 5R5.2, 5R6.2, 5R8.2, 5U1.12 (CSG), 5U1.19 (PGND), 5U1.7 (AGND), 6C1.2, 6C2.2, 6C3.2, 6C4.2, 6C5.2, 6D1.1 (K), 6D2.1 (K), 6D3.1 (K), 6D4.1 (K), 6J3.3 (Pin_3), 6J4.3 (Pin_3), 6J5.2 (Pin_2), 6U1.19 (TESTEN), 6U1.57 (GND), 6U2.8 (GND), 6U3.2 (GND)
- net I2C_SCL: now also 2R7.1, 2U1.13 (SCL), 4U1.26 (SCL), 6U1.7 (GPIO5)
- net I2C_SDA: now also 2R6.1, 2U1.12 (SDA), 4U1.27 (SDA), 6U1.6 (GPIO4)
- net ILIM_HIZ: now also 2R5.1, 2U1.6 (ILIM_HIZ)
- net IN_VALID: now also 3R1.1, 3U1.3 (EN), 6U1.13 (GPIO10)
- net N_ACN: now also 2Q1.3 (D), 2R1.2, 2U1.2 (ACN)
- net N_AF: now also 1D1.1 (A1), 1F1.2, 1R1.1, 1U1.1 (SENSE)
- net N_ALERT: now also 4R5.1, 4U1.25 (ALERT)
- net N_BOOT1: now also 5C2.1, 5U1.23 (BOOT1)
- net N_BOOT2: now also 5C3.1, 5U1.17 (BOOT2)
- net N_BTST1: now also 2C1.1, 2U1.30 (BTST1)
- net N_BTST2: now also 2C2.1, 2U1.25 (BTST2)
- net N_CBP: now also 2R3.2, 2R4.1, 2U1.18 (CELL_BATPRESZ)
- net N_CFETOFF: now also 4R7.1, 4U1.29 (CFETOFF)
- net N_CHG: now also 4Q1.1 (G), 4U1.45 (CHG)
- net N_CHGOK: now also 2R11.1, 2U1.4 (CHRG_OK)
- net N_COMP: now also 5C5.1, 5R6.1, 5U1.6 (COMP)
- net N_COMP1: now also 2R8.1, 2U1.16 (COMP1)
- net N_COMP1B: now also 2C5.1, 2R8.2
- net N_COMP2: now also 2C6.1, 2U1.17 (COMP2)
- net N_CP1: now also 4C5.1, 4U1.46 (CP1)
- net N_CS: now also 5Q2.2 (S), 5Q3.2 (S), 5R3.1, 5U1.13 (CS)
- net N_DFETOFF: now also 4R8.1, 4U1.30 (DFETOFF)
- net N_DITH: now also 5C7.1, 5U1.2 (DITH)
- net N_DSG: now also 4Q2.1 (G), 4U1.43 (DSG)
- net N_DVDD: now also 6C5.1, 6U1.23 (DVDD), 6U1.45 (VREG_VOUT)
- net N_EN: now also 5R7.2, 5R8.1, 5U1.26 (EN/UVLO)
- net N_FANPWM: now also 6J5.3 (Pin_3), 6U1.4 (GPIO2)
- net N_FANTACH: now also 6J5.4 (Pin_4), 6R8.1, 6U1.5 (GPIO3)
- net N_FB: now also 5R1.2, 5R2.1, 5U1.8 (FB)
- net N_G10: now also 5Q4.1 (G), 5U1.16 (HDRV2)
- net N_G3: now also 2Q1.1 (G), 2U1.31 (HIDRV1)
- net N_G4: now also 2Q2.1 (G), 2U1.29 (LODRV1)
- net N_G5: now also 2Q3.1 (G), 2U1.26 (LODRV2)
- net N_G6: now also 2Q4.1 (G), 2U1.24 (HIDRV2)
- net N_G7: now also 5Q1.1 (G), 5U1.24 (HDRV1)
- net N_G8: now also 5Q2.1 (G), 5U1.22 (LDRV1)
- net N_G9: now also 5Q3.1 (G), 5U1.18 (LDRV2)
- net N_GATE: now also 1Q1.1 (G), 1U1.10 (GATE)
- net N_IADPT: now also 2R9.1, 2U1.8 (IADPT)
- net N_IADPTB: now also 2C8.1, 2R9.2
- net N_IBAT: now also 2R10.1, 2U1.9 (IBAT)
- net N_IBATB: now also 2C9.1, 2R10.2
- net N_ISNS: now also 5U1.10 (ISNS-), 5U1.11 (ISNS+)
- net N_LED1: now also 6R2.1, 6U1.8 (GPIO6)
- net N_LED2: now also 6R3.1, 6U1.9 (GPIO7)
- net N_LED3: now also 6R4.1, 6U1.11 (GPIO8)
- net N_LED4: now also 6R5.1, 6U1.12 (GPIO9)
- net N_LEDA1: now also 6D1.2 (A), 6R2.2
- net N_LEDA2: now also 6D2.2 (A), 6R3.2
- net N_LEDA3: now also 6D3.2 (A), 6R4.2
- net N_LEDA4: now also 6D4.2 (A), 6R5.2
- net N_MODE: now also 5R5.1, 5U1.1 (MODE)
- net N_OV: now also 1R4.2, 1R5.1, 1U1.4 (OVLO)
- net N_PACKMID: now also 4Q1.2 (S), 4Q2.2 (S)
- net N_PGATE: now also 3Q1.1 (G), 3U1.5 (GATE)
- net N_PGD: now also 1R7.2, 1U1.8 (PGD)
- net N_PGOOD: now also 5R9.1, 5U1.14 (PGOOD)
- net N_PROCHOT: now also 2R12.1, 2U1.11 (PROCHOT)
- net N_PSYS: now also 2C7.1, 2U1.10 (PSYS)
- net N_PWR: now also 1R6.1, 1U1.7 (PWR)
- net N_QCLK: now also 6U1.51 (QSPI_SCLK), 6U2.2 (CLK)
- net N_QCS: now also 6U1.55 (QSPI_SS), 6U2.1 (CS)
- net N_QIO0: now also 6U1.52 (QSPI_SD0), 6U2.3 (IO0)
- net N_QIO1: now also 6U1.54 (QSPI_SD1), 6U2.4 (IO1)
- net N_QIO2: now also 6U1.53 (QSPI_SD2), 6U2.5 (IO2)
- net N_QIO3: now also 6U1.50 (QSPI_SD3), 6U2.6 (IO3)
- net N_REG1: now also 4C3.1, 4R7.2, 4R8.2, 4U1.35 (REG1)
- net N_REG18: now also 4C1.1, 4U1.24 (REG18)
- net N_REG2: now also 4C2.1, 4U1.34 (REG2)
- net N_RST: now also 4R6.1, 4U1.33 (RST_SHUT)
- net N_RT: now also 5R4.1, 5U1.3 (RT/SYNC)
- net N_RUN: now also 6R1.1, 6U1.26 (RUN)
- net N_SLOPE: now also 5C6.1, 5U1.4 (SLOPE)
- net N_SS: now also 5C4.1, 5U1.5 (SS)
- net N_SWCLK: now also 6J4.1 (Pin_1), 6U1.24 (SWCLK)
- net N_SWDIO: now also 6J4.2 (Pin_2), 6U1.25 (SWDIO)
- net N_TMR: now also 1C1.1, 1U1.6 (TIMER)
- net N_USBDM: now also 6R6.1, 6U1.46 (USB_DM)
- net N_USBDM_C: now also 6J3.1 (Pin_1), 6R6.2
- net N_USBDP: now also 6R7.1, 6U1.47 (USB_DP)
- net N_USBDP_C: now also 6J3.2 (Pin_2), 6R7.2
- net N_UV: now also 1R2.2, 1R3.1, 1U1.3 (UVLO)
- net N_VCAP: now also 3C1.1, 3U1.1 (VCAP)
- net N_XIN: now also 6C1.1, 6U1.20 (XIN), 6Y1.1
- net N_XOUT: now also 6C2.1, 6U1.21 (XOUT), 6Y1.2
- net PACK+: now also 4C4.1, 4C5.2, 4J6.1 (Pin_1), 4Q1.3 (D), 4U1.36 (REGIN), 4U1.47 (BAT)
- net REGN: now also 2C3.1, 2U1.28 (REGN)
- net SW1: now also 2C1.2, 2L1.1, 2Q1.2 (S), 2Q2.3 (D), 2U1.32 (SW1)
- net SW1_OUT: now also 5C2.2, 5L1.1, 5Q1.2 (S), 5Q2.3 (D), 5U1.25 (SW1)
- net SW2: now also 2C2.2, 2L1.2, 2Q3.3 (D), 2Q4.2 (S), 2U1.23 (SW2)
- net SW2_OUT: now also 5C3.2, 5L1.2, 5Q3.3 (D), 5Q4.2 (S), 5U1.15 (SW2)
- net TS1: now also 4R2.1, 4U1.21 (TS1)
- net TS2: now also 4R3.1, 4U1.22 (TS2)
- net TS3: now also 4R4.1, 4U1.23 (TS3)
- net VBAT: now also 2R2.2, 2U1.19 (SRN), 3C1.2, 3Q1.2 (S), 3U1.6 (ANODE), 4Q2.3 (D)
- net VBUS: now also 2R1.1, 2U1.1 (VBUS), 2U1.3 (ACP)
- net VC0: now also 4C6.1, 4R9.2, 4U1.16 (VC0)
- net VC1: now also 4C7.1, 4R10.2, 4U1.15 (VC1)
- net VC2: now also 4C8.1, 4R11.2, 4U1.14 (VC2)
- net VC3: now also 4C9.1, 4R12.2, 4U1.13 (VC3)
- net VC4: now also 4C10.1, 4R13.2, 4U1.12 (VC4)
- net VCC: now also 5C8.1, 5U1.20 (VCC), 5U1.21 (BIAS)
- net VDDA: now also 2C4.1, 2R3.1, 2U1.7 (VDDA)
- net VIN_LM: now also 1Q1.3 (D), 1R1.2, 1R2.1, 1R4.1, 1U1.2 (VIN)
- net VIN_SYS: now also 1Q1.2 (S), 1U1.9 (OUT), 3C2.1, 3C3.1, 3Q1.3 (D), 3U1.4 (CATHODE), 5C1.1, 5Q1.3 (D), 5R7.1, 5U1.27 (VIN), 5U1.28 (VISNS), 6C3.1, 6U3.1 (VIN), 6U3.3 (EN)
- net VOUT12: now also 5C10.1, 5C9.1, 5J2.1 (Pin_1), 5Q4.3 (D), 5R1.1, 5U1.9 (VOSNS), 6J5.1 (Pin_1)
- net VSYS: now also 2Q4.3 (D), 2R2.1, 2U1.20 (SRP), 2U1.22 (VSYS)

Commit message: fix part selection
Parts:
- 1F1: footprint Fuse:Fuse_1206_3216Metric -> Fuse:Fuse_Blade_ATO_directSolder
- 1R1, 2R1, 2R2, 4R1, 5R3: footprint Resistor_SMD:R_2512_6332Metric -> Resistor_SMD:R_Shunt_Vishay_WSR2_WSR3
Changed lines of the file:
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@@
       (effects (font (size 1.27 1.27)))
     )
-    (property "Footprint" "Fuse:Fuse_1206_3216Metric" (at 63.5 39.37 0)
+    (property "Footprint" "Fuse:Fuse_Blade_ATO_directSolder" (at 63.5 39.37 0)
       (effects (font (size 1.0 1.0)) hide)
     )
@@
       (effects (font (size 1.27 1.27)))
     )
-    (property "Footprint" "Resistor_SMD:R_2512_6332Metric" (at 114.3 39.37 0)
+    (property "Footprint" "Resistor_SMD:R_Shunt_Vishay_WSR2_WSR3" (at 114.3 39.37 0)
       (effects (font (size 1.0 1.0)) hide)
     )
@@
       (effects (font (size 1.27 1.27)))
     )
-    (property "Footprint" "Resistor_SMD:R_2512_6332Metric" (at 165.1 45.72 0)
+    (property "Footprint" "Resistor_SMD:R_Shunt_Vishay_WSR2_WSR3" (at 165.1 45.72 0)
       (effects (font (size 1.0 1.0)) hide)
     )
@@
       (effects (font (size 1.27 1.27)))
     )
-    (property "Footprint" "Resistor_SMD:R_2512_6332Metric" (at 165.1 71.12 0)
+    (property "Footprint" "Resistor_SMD:R_Shunt_Vishay_WSR2_WSR3" (at 165.1 71.12 0)
       (effects (font (size 1.0 1.0)) hide)
     )
@@
       (effects (font (size 1.27 1.27)))
     )
-    (property "Footprint" "Resistor_SMD:R_2512_6332Metric" (at 381.0 147.32 0)
+    (property "Footprint" "Resistor_SMD:R_Shunt_Vishay_WSR2_WSR3" (at 381.0 147.32 0)
       (effects (font (size 1.0 1.0)) hide)
     )
@@
       (effects (font (size 1.27 1.27)))
     )
-    (property "Footprint" "Resistor_SMD:R_2512_6332Metric" (at 431.8 147.32 0)
-      (effects (font (size 1.0 1.0)) hide)
-    )
+    (property "Footprint" "Resistor_SMD:R_Shunt_Vishay_WSR2_WSR3" (at 431.8 147.32 0)
+      (effects (font (size 1.0 1.0)) hide)
+    )

Commit message: new terminal power rating metric, new FET selection
Parts:
- 1Q1, 3Q1, 4Q1, 4Q2: value N-FET 40V -> NTMFS5C410N; footprint Package_TO_SOT_SMD:TO-252-2 -> Package_SON:VSONP-8-1EP_5x6_P1.27mm; symbol Transistor_FET:Q_NMOS_GSD -> Transistor_FET:Q_NMOS_SGD
- 2Q1, 2Q2, 2Q3, 2Q4: value N-FET 30V -> NTMFS4C01N; footprint Package_TO_SOT_SMD:TO-252-2 -> Package_SON:VSONP-8-1EP_5x6_P1.27mm; symbol Transistor_FET:Q_NMOS_GSD -> Transistor_FET:Q_NMOS_SGD
- 5Q1, 5Q2, 5Q3, 5Q4: value N-FET 40V -> NTMFS5C430N; footprint Package_TO_SOT_SMD:TO-252-2 -> Package_SON:VSONP-8-1EP_5x6_P1.27mm; symbol Transistor_FET:Q_NMOS_GSD -> Transistor_FET:Q_NMOS_SGD
Connections:
- net GND: now also 2Q2.1 (S), 2Q3.1 (S); no longer 2Q2.2 (S), 2Q3.2 (S)
- net N_CHG: now also 4Q1.2 (G); no longer 4Q1.1 (G)
- net N_CS: now also 5Q2.1 (S), 5Q3.1 (S); no longer 5Q2.2 (S), 5Q3.2 (S)
- net N_DSG: now also 4Q2.2 (G); no longer 4Q2.1 (G)
- net N_G10: now also 5Q4.2 (G); no longer 5Q4.1 (G)
- net N_G3: now also 2Q1.2 (G); no longer 2Q1.1 (G)
- net N_G4: now also 2Q2.2 (G); no longer 2Q2.1 (G)
- net N_G5: now also 2Q3.2 (G); no longer 2Q3.1 (G)
- net N_G6: now also 2Q4.2 (G); no longer 2Q4.1 (G)
- net N_G7: now also 5Q1.2 (G); no longer 5Q1.1 (G)
- net N_G8: now also 5Q2.2 (G); no longer 5Q2.1 (G)
- net N_G9: now also 5Q3.2 (G); no longer 5Q3.1 (G)
- net N_GATE: now also 1Q1.2 (G); no longer 1Q1.1 (G)
- net N_PACKMID: now also 4Q1.1 (S), 4Q2.1 (S); no longer 4Q1.2 (S), 4Q2.2 (S)
- net N_PGATE: now also 3Q1.2 (G); no longer 3Q1.1 (G)
- net SW1: now also 2Q1.1 (S); no longer 2Q1.2 (S)
- net SW1_OUT: now also 5Q1.1 (S); no longer 5Q1.2 (S)
- net SW2: now also 2Q4.1 (S); no longer 2Q4.2 (S)
- net SW2_OUT: now also 5Q4.1 (S); no longer 5Q4.2 (S)
- net VBAT: now also 3Q1.1 (S); no longer 3Q1.2 (S)
- net VIN_SYS: now also 1Q1.1 (S); no longer 1Q1.2 (S)

Commit message: board fixup, added shunt sense gate
Connections:
- net VBUS is gone; now on net VIN_SYS: 2R1.1, 2U1.1 (VBUS), 2U1.3 (ACP)
Changed lines of the file:
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@@
     (effects (font (size 1.27 1.27)))
   )
-  (label "VBUS" (at 175.26 26.669999999999998 0)
+  (label "VIN_SYS" (at 175.26 26.669999999999998 0)
     (effects (font (size 1.27 1.27)))
   )
-  (label "VBUS" (at 165.1 41.91 0)
+  (label "VIN_SYS" (at 165.1 41.91 0)
     (effects (font (size 1.27 1.27)))
   )
-  (label "VBUS" (at 175.26 31.75 0)
+  (label "VIN_SYS" (at 175.26 31.75 0)
     (effects (font (size 1.27 1.27)))
   )
